File: ROBOT_2_PCB/ROBOT_2_PCB.kicad_pcb (KiCad board)
At the start: 2 copper layers, 18 parts, among them J1 Conn_01x04, J2 Conn_01x02, J3 Conn_01x02, J4 DB15_Female, J5 Conn_01x01_Female, U1 ULN2003

Commit message: r2 pcb created
Parts:
- removed BT1: Conn_01x04, modfiles:bluetooth
- added C1: 104nF, modfiles:Capacitor_Disc_Small, F.Cu at (150.9, 58.4)
- added C2: 104nF, modfiles:Capacitor_Disc_Small, F.Cu at (71.6, 64.8)
- added J1: Bluetooth, Connector_PinHeader_2.54mm:PinHeader_2x04_P2.54mm_Vertical, F.Cu at (44.1, 73.2)
- moved GPIO_PINS_INPUT1 156.7 mm to (216.8, 66.6), turned to -90 degrees
- moved GPIO_PINS_OUTPUT1 140.1 mm to (223.4, 87.7), turned to -90 degrees
- moved db-2 75.5 mm to (145.2, 138.7), turned to 180 degrees
- moved NEPAL1 41.0 mm to (47.3, 34.7)
- moved R4 36.0 mm to (190.4, 101.2), turned to -90 degrees
- moved R3 35.6 mm to (185.6, 101.2), turned to -90 degrees
- moved U1 29.9 mm to (224.3, 48.2)
- moved S1 29.6 mm to (102.6, 76.9)
- moved S2 29.4 mm to (177.4, 77.2)
- moved PN-2 29.3 mm to (177.7, 137.4)
- moved R2 29.1 mm to (195.2, 101.4)
- moved db-3 28.8 mm to (225.6, 114.6)
- moved MPU1 28.8 mm to (232.6, 46.7)
- moved PN-1 28.3 mm to (188.1, 137.4)
- moved R1 28.3 mm to (180.6, 108.8)
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- renumbered J1 to MPU1, J5 to NEPAL1, J2 to PN-1, J3 to PN-2, Encoders1 to db-1, J4 to db-2, DIR_PWM1 to db-3
Connections:
- GPIO_PINS_INPUT1 pad 1: GPIO_INPUT_1 -> I1
- GPIO_PINS_INPUT1 pad 2: GPIO_INPUT_2 -> I2
- GPIO_PINS_INPUT1 pad 3: GPIO_INPUT_3 -> I3
- GPIO_PINS_INPUT1 pad 4: GPIO_INPUT_4 -> I4
- GPIO_PINS_INPUT1 pad 5: GPIO_INPUT_5 -> I5
- GPIO_PINS_OUTPUT1 pad 1: GPIO_OUTPUT_1 -> O1
- GPIO_PINS_OUTPUT1 pad 2: GPIO_OUTPUT_2 -> O2
- GPIO_PINS_OUTPUT1 pad 3: GPIO_OUTPUT_3 -> O3
- GPIO_PINS_OUTPUT1 pad 4: GPIO_OUTPUT_4 -> O4
- GPIO_PINS_OUTPUT1 pad 5: GPIO_OUTPUT_5 -> O5
- MPU1 pad 1: 5V -> 5VS
- S1 pad 1: unconnected-(S1-Pad1) -> GND
- S1 pad 18: Motor_3_Enc_1 -> unconnected-(S1-Pad18)
- S1 pad 38: GPIO_INPUT_1 -> unconnected-(S1-Pad38)
- S1 pad 40: GPIO_INPUT_2 -> unconnected-(S1-Pad40)
- S1 pad 41: GPIO_INPUT_4 -> unconnected-(S1-Pad41)
- S1 pad 42: GPIO_INPUT_3 -> unconnected-(S1-Pad42)
- S1 pad 43: GPIO_INPUT_5 -> unconnected-(S1-Pad43)
- S1 pad 49: unconnected-(S1-Pad49) -> GND
- S1 pad 50: unconnected-(S1-Pad50) -> GND
- S1 pad 51: unconnected-(S1-Pad51) -> GND
- S1 pad 52: unconnected-(S1-Pad52) -> GND
- S1 pad 53: 5V -> unconnected-(S1-Pad53)
- S1 pad 54: 5V -> unconnected-(S1-Pad54)
- S1 pad 73: MPU_SCL -> unconnected-(S1-Pad73)
- S1 pad 74: MPU_SDA -> unconnected-(S1-Pad74)
- S1 pad 79: unconnected-(S1-Pad79) -> BT_TX
- S1 pad 80: unconnected-(S1-Pad80) -> BT_RX
- S1 pad 90: Motor_2_Enc_1 -> unconnected-(S1-Pad90)
- S1 pad 91: Motor_3_DIR -> unconnected-(S1-Pad91)
- S1 pad 92: Motor_4_DIR -> unconnected-(S1-Pad92)
- S1 pad 93: Motor_1_DIR -> unconnected-(S1-Pad93)
- S1 pad 94: Motor_2_DIR -> unconnected-(S1-Pad94)
- S1 pad 96: Motor_4_Pwm -> unconnected-(S1-Pad96)
- S1 pad 97: Motor_1_Pwm -> Motor_3_Enc_1
- S1 pad 98: Motor_2_Pwm -> unconnected-(S1-Pad98)
- S2 pad 1: unconnected-(S2-Pad1) -> GND
- S2 pad 13: BT_RX -> Motor_4_Pwm
- S2 pad 14: BT_TX -> Motor_2_DIR
- S2 pad 21: unconnected-(S2-Pad21) -> Picker_Motor2_E2
- S2 pad 22: unconnected-(S2-Pad22) -> Picker_Motor2_E1
- S2 pad 31: unconnected-(S2-Pad31) -> Motor_1_Pwm
- S2 pad 32: unconnected-(S2-Pad32) -> Motor_2_Pwm
- S2 pad 36: unconnected-(S2-Pad36) -> Picker_Motor1_DIR
- S2 pad 38: unconnected-(S2-Pad38) -> Vertical_Motor_DIR
- S2 pad 40: unconnected-(S2-Pad40) -> Motor_1_DIR
- S2 pad 41: GPIO_OUTPUT_1 -> unconnected-(S2-Pad41)
- S2 pad 42: GPIO_OUTPUT_5 -> Motor_3_DIR
- S2 pad 43: GPIO_OUTPUT_2 -> unconnected-(S2-Pad43)
- S2 pad 44: Picker_Motor2_E1 -> Horizontal_Motor_DIR
- S2 pad 45: Picker_Motor2_E2 -> unconnected-(S2-Pad45)
- S2 pad 46: GPIO_OUTPUT_4 -> Picker_Motor2_DIR
- S2 pad 47: GPIO_OUTPUT_3 -> unconnected-(S2-Pad47)
- S2 pad 51: unconnected-(S2-Pad51) -> GND
- S2 pad 52: unconnected-(S2-Pad52) -> GND
- S2 pad 58: unconnected-(S2-Pad58) -> I1
- S2 pad 60: unconnected-(S2-Pad60) -> I2
- S2 pad 62: unconnected-(S2-Pad62) -> I3
- S2 pad 64: unconnected-(S2-Pad64) -> I4
- S2 pad 66: unconnected-(S2-Pad66) -> I5
- S2 pad 73: unconnected-(S2-Pad73) -> MPU_SCL
- S2 pad 74: unconnected-(S2-Pad74) -> MPU_SDA
- S2 pad 76: unconnected-(S2-Pad76) -> O1
- S2 pad 78: unconnected-(S2-Pad78) -> O2
- S2 pad 80: unconnected-(S2-Pad80) -> O3
- S2 pad 82: unconnected-(S2-Pad82) -> O4
- S2 pad 84: unconnected-(S2-Pad84) -> O5
- S2 pad 91: Picker_Motor1_DIR -> unconnected-(S2-Pad91)
- S2 pad 92: Picker_Motor2_DIR -> unconnected-(S2-Pad92)
- S2 pad 93: Horizontal_Motor_DIR -> Motor_4_DIR
- S2 pad 94: Vertical_Motor_DIR -> unconnected-(S2-Pad94)
- db-1 pad 1: FW4_E1 -> Motor_4_Enc_1
- db-1 pad 10: Motor_1_Pwm -> Motor_2_Enc_1
- db-1 pad 11: Motor_2_Pwm -> Motor_2_Enc_2
- db-1 pad 12: Motor_4_Pwm -> FW2_E2
- db-1 pad 13: Vertical_Motor_E2 -> Motor_3_Enc_2
- db-1 pad 14: Picker_Motor1_E2 -> FW3_E2
- db-1 pad 15: unconnected-(Encoders1-Pad15) -> FW3_E1
- db-1 pad 2: Motor_4_Enc_2 -> FW4_E1
- db-1 pad 3: Motor_1_Enc_2 -> FW4_E2
- db-1 pad 4: Motor_1_Enc_1 -> Motor_4_Enc_2
- db-1 pad 5: Motor_3_Enc_1 -> FW1_E1
- db-1 pad 6: Motor_3_Enc_2 -> Motor_1_Enc_2
- db-1 pad 7: Motor_2_Enc_2 -> Motor_1_Enc_1
- db-1 pad 8: unconnected-(Encoders1-Pad8) -> FW1_E2
- db-1 pad 9: Motor_3_Pwm -> FW2_E1
- db-2 pad 1: FW1_E1 -> Horizontal_Motor_DIR
- db-2 pad 10: FW2_E2 -> Motor_1_DIR
- db-2 pad 11: FW3_E2 -> Motor_3_Pwm
- db-2 pad 12: FW4_E2 -> Motor_3_Enc_1
- db-2 pad 13: unconnected-(J4-Pad13) -> Vertical_Motor_E2
- db-2 pad 14: unconnected-(J4-Pad14) -> Motor_4_Pwm
- db-2 pad 15: unconnected-(J4-Pad15) -> Picker_Motor1_E2
- db-2 pad 2: FW2_E1 -> Picker_Motor2_DIR
- db-2 pad 3: FW3_E1 -> unconnected-(db-2-Pad3)
- db-2 pad 4: unconnected-(J4-Pad4) -> Motor_1_Pwm
- db-2 pad 5: unconnected-(J4-Pad5) -> Horizontal_Motor_E2
- db-2 pad 7: unconnected-(J4-Pad7) -> Horizontal_Motor_E1
- db-2 pad 8: unconnected-(J4-Pad8) -> Picker_Motor2_E2
- db-2 pad 9: FW1_E2 -> Motor_3_DIR
- db-3 pad 1: Picker_Motor2_E1 -> GND
- db-3 pad 10: Picker_Motor1_E1 -> Vertical_Motor_DIR
- db-3 pad 11: unconnected-(DIR_PWM1-Pad11) -> Picker_Motor1_DIR
- db-3 pad 12: Vertical_Motor_E1 -> Motor_2_Pwm
- db-3 pad 13: unconnected-(DIR_PWM1-Pad13) -> Picker_Motor2_E1
- db-3 pad 14: Picker_Motor1_DIR -> Picker_Motor1_E1
- db-3 pad 15: Horizontal_Motor_DIR -> Motor_2_DIR
- db-3 pad 2: Horizontal_Motor_E1 -> Picker_Motor2_PWM
- db-3 pad 3: Picker_Motor2_DIR -> Vertical_Motor_PWM
- db-3 pad 4: Vertical_Motor_DIR -> Horizontal_Motor_PWM
- db-3 pad 5: Picker_Motor2_PWM -> Picker_Motor1_PWM
- db-3 pad 6: Vertical_Motor_PWM -> Motor_4_DIR
- db-3 pad 7: Horizontal_Motor_PWM -> unconnected-(db-3-Pad7)
- db-3 pad 8: Picker_Motor1_PWM -> Vertical_Motor_E1
- db-3 pad 9: Picker_Motor2_E2 -> GND
Routing:
- net 12V: track 0.00 -> 202.6 mm
- net STM1_RX: track 0.00 -> 177.5 mm, vias 0 -> 4
- net STM1_TX: track 0.00 -> 164.0 mm, vias 0 -> 4
- net 5V: track 0.00 -> 163.0 mm
- net Vertical_Motor_DIR: track 0.00 -> 162.1 mm
- net Picker_Motor1_DIR: track 0.61 -> 156.9 mm
- net Motor_2_Pwm: track 0.00 -> 155.0 mm
- net Picker_Motor2_E1: track 0.00 -> 153.3 mm
- net Picker_Motor1_E1: track 0.00 -> 148.2 mm
- net Motor_2_DIR: track 0.00 -> 135.8 mm
- net Vertical_Motor_E1: track 0.00 -> 130.3 mm
- net PN_01: track 0.00 -> 119.8 mm
- net PN_02: track 0.00 -> 119.5 mm
- net Vertical_Motor_E2: track 0.00 -> 114.6 mm
- net Motor_4_Pwm: track 0.00 -> 104.5 mm
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Other:
- board text added: "#AARJAN"
- board text added: "12V"
- board text added: "3.3V"
- board text added: "5A"
- board text added: "5V"
- board text added: "FW1E1"
- board text added: "FW1E2"
- board text added: "FW2E1"
- board text added: "FW2E2"
- board text added: "FW3E1"
- board text added: "FW3E2"
- board text added: "FW4E1"
- board text added: "FW4E2"
- board text added: "GND"
- board text added: "GPIO_INPUT_PINS"
- board text added: "HMD"
- board text added: "HME1"
- board text added: "HME2"
- board text added: "HMP"
- board text added: "M1D"
- board text added: "M1E1"
- board text added: "M1E2"
- board text added: "M1P"
- board text added: "M2D"
- board text added: "M2E1"
- board text added: "M2E2"
- board text added: "M2P"
- board text added: "M3D"
- board text added: "M3E1"
- board text added: "M3E2"
- board text added: "M3P"
- board text added: "M4D"
- board text added: "M4E1"
- board text added: "M4E2"
- board text added: "M4P"
- board text added: "N"
- board text added: "PM1D"
- board text added: "PM1E1"
- board text added: "PM1E2"
- board text added: "PM1P"
- board text added: "PM2D"
- board text added: "PM2E1"
- board text added: "PM2E2"
- board text added: "PM2P"
- board text added: "VMD"
- board text added: "VME1"
- board text added: "VME2"
- board text added: "VMP"
- board text removed: "#RJN"

Commit message: Finally created
Parts:
- added C3: 104nF, modfiles:Capacitor_Disc_Small, F.Cu at (41.1, 70.1)
- added D1: LED, modfiles:LED_D3.0mm, F.Cu at (67.3, 61.5)
- added D2: LED, modfiles:LED_D3.0mm, F.Cu at (142.2, 62.7)
- added D3: LED, modfiles:LED_D3.0mm, F.Cu at (239.6, 75.0)
- added D4: LED, modfiles:LED_D3.0mm, F.Cu at (228.6, 50.0)
- added D5: LED, modfiles:LED_D3.0mm, F.Cu at (228.6, 40.9)
- added MPU1: 330, modfiles:Resistor_small, F.Cu at (231.9, 73.5)
- added S1I1: 330, modfiles:Resistor_small, F.Cu at (85.3, 61.5)
- added S2I1: 330, modfiles:Resistor_small, F.Cu at (141.2, 77.2)
- added pneu1: 1K, modfiles:Resistor_small, F.Cu at (228.3, 36.1)
- added pneu2: 1K, modfiles:Resistor_small, F.Cu at (222.8, 56.1)
- moved PN-1 103.4 mm to (239.0, 47.5), turned to 90 degrees
- moved PN-2 99.6 mm to (238.9, 58.9), turned to 90 degrees
- moved IMU1 43.5 mm to (239.3, 89.7)
- moved U1 20.1 mm to (215.4, 30.2), turned to 0 degrees
- moved NEPAL1 1.62 mm to (48.9, 34.6)
- renumbered GPIO_PINS_INPUT1 to GPIO_INPUT_PINS1, GPIO_PINS_OUTPUT1 to GPIO_OUTPUT_PINS1, MPU1 to IMU1
Connections:
- PN-1 pad 1: +12V -> 12V
- PN-2 pad 1: +12V -> 12V
- S1 pad 49: GND -> Net-(S1-Pad49)
- S1 pad 50: GND -> Net-(S1-Pad49)
Routing:
- net PN_01: track 119.8 -> 22.0 mm
- net 12V: track 202.6 -> 285.1 mm
- net PN_02: track 119.5 -> 39.4 mm
- net 5V: track 163.0 -> 207.8 mm
- net MPU_SDA: track 72.3 -> 38.7 mm
- net Net-(S1I1-Pad2): track 0.00 -> 31.5 mm
- net 5VS: track 40.3 -> 64.2 mm
- net GND: track 45.2 -> 24.6 mm, vias 4 -> 2
- net MPU_SCL: track 70.1 -> 51.5 mm
- net +12V: track 13.3 -> 0.00 mm
- net Net-(D3-Pad1): track 0.00 -> 12.3 mm
- net Net-(pneu1-Pad2): track 0.00 -> 11.4 mm
- net Net-(D2-Pad1): track 0.00 -> 7.28 mm
- net Net-(pneu2-Pad2): track 0.00 -> 6.83 mm
- net Net-(R1-Pad2): track 91.1 -> 95.6 mm
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Other:
- board text added: "1K"
- board text added: "330"
- board text added: "B3"
- board text added: "B5"
- board text added: "C13"
- board text added: "C15"
- board text added: "D2"
- board text added: "D4"
- board text added: "D6"
- board text added: "E3"
- board text added: "E5"
- board text added: "G"
- board text added: "GI"
- board text added: "GO"
- board text added: "H1"
- board text added: "IMU"
- board text added: "SCL"
- board text added: "SDA"
- board text added: "ST_1"
- board text added: "ST_2"
- board text added: "TEAM NEPAL"
- board text added: "X"
- board text removed: "GND"
- board text removed: "GPIO_INPUT_PINS"

Commit message: Finally Created1
Parts:
- moved S1I1 10.7 mm to (96.0, 60.2)
- moved db-1 10.1 mm to (46.5, 138.2)
- moved db-3 9.39 mm to (233.5, 119.8)
- moved db-2 7.47 mm to (145.6, 146.1)
- moved NEPAL1 1.40 mm to (47.5, 34.5)
Connections:
- db-1 pad 1: Motor_4_Enc_1 -> Motor_4_Enc_2
- db-1 pad 10: Motor_2_Enc_1 -> FW4_E1
- db-1 pad 11: Motor_2_Enc_2 -> Motor_4_Enc_1
- db-1 pad 12: FW2_E2 -> FW2_E1
- db-1 pad 13: Motor_3_Enc_2 -> Motor_2_Enc_1
- db-1 pad 14: FW3_E2 -> Motor_2_Enc_2
- db-1 pad 15: FW3_E1 -> FW2_E2
- db-1 pad 2: FW4_E1 -> FW1_E1
- db-1 pad 3: FW4_E2 -> Motor_1_Enc_2
- db-1 pad 4: Motor_4_Enc_2 -> Motor_1_Enc_1
- db-1 pad 5: FW1_E1 -> FW1_E2
- db-1 pad 6: Motor_1_Enc_2 -> FW3_E1
- db-1 pad 7: Motor_1_Enc_1 -> FW3_E2
- db-1 pad 8: FW1_E2 -> Motor_3_Enc_2
- db-1 pad 9: FW2_E1 -> FW4_E2
Routing:
- net Motor_4_Enc_1: track 43.0 -> 88.1 mm
- net FW4_E1: track 36.3 -> 75.5 mm
- net FW4_E2: track 24.3 -> 45.9 mm
- net FW1_E1: track 35.5 -> 55.8 mm
- net Motor_1_Enc_2: track 35.8 -> 55.4 mm
- net Picker_Motor1_PWM: track 39.4 -> 58.1 mm
- net Horizontal_Motor_PWM: track 33.6 -> 52.1 mm
- net Motor_4_DIR: track 45.8 -> 64.1 mm
- net Motor_2_Pwm: track 155.9 -> 138.1 mm
- net Motor_1_Enc_1: track 35.6 -> 53.4 mm
- net FW1_E2: track 49.1 -> 66.8 mm
- net Motor_4_Enc_2: track 24.9 -> 41.2 mm
- net Picker_Motor1_DIR: track 157.8 -> 143.2 mm
- net Picker_Motor2_E1: track 154.2 -> 140.1 mm
- net FW3_E1: track 45.2 -> 58.9 mm
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
Commit message: Finally Created
Routing:
- net STM1_TX: track 164.0 -> 178.1 mm
- net FW1_E1: track 55.8 -> 48.6 mm
- net Motor_1_Enc_2: track 55.4 -> 48.5 mm
- net GND: track 23.2 -> 29.0 mm
- net Motor_1_Enc_1: track 53.4 -> 48.1 mm
- net Motor_4_Enc_2: track 41.2 -> 38.5 mm
- net FW4_E2: track 45.9 -> 43.2 mm
- net Motor_3_Enc_2: track 55.2 -> 52.6 mm
- net FW3_E1: track 58.9 -> 56.3 mm
- net FW3_E2: track 53.6 -> 52.1 mm
- net FW2_E1: track 93.7 -> 94.9 mm
- net FW1_E2: track 66.8 -> 65.8 mm
- net 5VS: track 64.2 -> 64.8 mm
Other:
- board text added: "2003"
- board text removed: "N"

Commit message: Redesigning in process
Connections:
- S1 pad 13: FW2_E2 -> Motor_4_Pwm
- S1 pad 14: FW2_E1 -> Motor_3_Pwm
- S1 pad 15: unconnected-(S1-Pad15) -> FW1_E1
- S1 pad 17: Motor_3_Enc_2 -> FW2_E2
- S1 pad 18: unconnected-(S1-Pad18) -> FW2_E1
- S1 pad 21: FW3_E2 -> unconnected-(S1-Pad21)
- S1 pad 22: FW3_E1 -> unconnected-(S1-Pad22)
- S1 pad 31: FW1_E1 -> Motor_1_Pwm
- S1 pad 32: FW1_E2 -> Motor_2_Pwm
- S1 pad 41: unconnected-(S1-Pad41) -> M3D
- S1 pad 43: unconnected-(S1-Pad43) -> M2D
- S1 pad 46: FW4_E1 -> unconnected-(S1-Pad46)
- S1 pad 47: FW4_E2 -> M1D
- S1 pad 95: Motor_3_Pwm -> M4D
- S1 pad 98: unconnected-(S1-Pad98) -> Motor_3_Enc_2
- S2 pad 13: Motor_4_Pwm -> Picker_Motor2_PWM
- S2 pad 14: Motor_2_DIR -> Picker_Motor1_PWM
- S2 pad 21: Picker_Motor2_E2 -> unconnected-(S2-Pad21)
- S2 pad 22: Picker_Motor2_E1 -> unconnected-(S2-Pad22)
- S2 pad 31: Motor_1_Pwm -> Horizontal_Motor_PWM
- S2 pad 32: Motor_2_Pwm -> Vertical_Motor_PWM
- S2 pad 40: Motor_1_DIR -> unconnected-(S2-Pad40)
- S2 pad 42: Motor_3_DIR -> unconnected-(S2-Pad42)
- S2 pad 45: unconnected-(S2-Pad45) -> Picker_Motor2_E2
- S2 pad 69: unconnected-(S2-Pad69) -> MPU_SCL
- S2 pad 73: MPU_SCL -> Picker_Motor2_E1
- S2 pad 78: O2 -> FW3_E1
- S2 pad 80: O3 -> O2
- S2 pad 82: O4 -> O3
- S2 pad 84: O5 -> O4
- S2 pad 86: unconnected-(S2-Pad86) -> O5
- S2 pad 93: Motor_4_DIR -> unconnected-(S2-Pad93)
- S2 pad 95: Picker_Motor1_PWM -> unconnected-(S2-Pad95)
- S2 pad 96: Picker_Motor2_PWM -> unconnected-(S2-Pad96)
- S2 pad 97: Horizontal_Motor_PWM -> FW4_E2
- S2 pad 98: Vertical_Motor_PWM -> FW4_E1
- db-1 pad 1: Motor_4_Enc_2 -> M2D
- db-1 pad 10: FW4_E1 -> M1D
- db-1 pad 12: FW2_E1 -> Motor_2_Enc_1
- db-1 pad 13: Motor_2_Enc_1 -> Motor_2_Enc_2
- db-1 pad 14: Motor_2_Enc_2 -> Motor_4_Pwm
- db-1 pad 15: FW2_E2 -> FW1_E1
- db-1 pad 2: FW1_E1 -> M3D
- db-1 pad 3: Motor_1_Enc_2 -> Motor_1_Pwm
- db-1 pad 4: Motor_1_Enc_1 -> Motor_1_Enc_2
- db-1 pad 5: FW1_E2 -> Motor_1_Enc_1
- db-1 pad 6: FW3_E1 -> Motor_2_Pwm
- db-1 pad 7: FW3_E2 -> FW2_E1
- db-1 pad 8: Motor_3_Enc_2 -> FW2_E2
- db-1 pad 9: FW4_E2 -> Motor_4_Enc_2
- db-2 pad 1: Horizontal_Motor_DIR -> Picker_Motor2_DIR
- db-2 pad 10: Motor_1_DIR -> unconnected-(db-2-Pad10)
- db-2 pad 11: Motor_3_Pwm -> unconnected-(db-2-Pad11)
- db-2 pad 12: Motor_3_Enc_1 -> M4D
- db-2 pad 13: Vertical_Motor_E2 -> Motor_3_Enc_1
- db-2 pad 14: Motor_4_Pwm -> Motor_3_Enc_2
- db-2 pad 15: Picker_Motor1_E2 -> FW1_E2
- db-2 pad 2: Picker_Motor2_DIR -> Picker_Motor2_E2
- db-2 pad 3: unconnected-(db-2-Pad3) -> Horizontal_Motor_PWM
- db-2 pad 4: Motor_1_Pwm -> Horizontal_Motor_E2
- db-2 pad 5: Horizontal_Motor_E2 -> Horizontal_Motor_E1
- db-2 pad 6: unconnected-(db-2-Pad6) -> Picker_Motor1_E2
- db-2 pad 7: Horizontal_Motor_E1 -> Picker_Motor2_PWM
- db-2 pad 8: Picker_Motor2_E2 -> Vertical_Motor_E2
- db-2 pad 9: Motor_3_DIR -> unconnected-(db-2-Pad9)
- db-3 pad 12: Motor_2_Pwm -> unconnected-(db-3-Pad12)
- db-3 pad 15: Motor_2_DIR -> unconnected-(db-3-Pad15)
- db-3 pad 2: Picker_Motor2_PWM -> unconnected-(db-3-Pad2)
- db-3 pad 3: Vertical_Motor_PWM -> unconnected-(db-3-Pad3)
- db-3 pad 4: Horizontal_Motor_PWM -> unconnected-(db-3-Pad4)
- db-3 pad 6: Motor_4_DIR -> unconnected-(db-3-Pad6)
Routing:
- net Vertical_Motor_DIR: track 149.4 -> 0.00 mm
- net Picker_Motor1_DIR: track 143.2 -> 0.00 mm
- net Motor_2_DIR: track 124.4 -> 0.00 mm
- net Picker_Motor1_E1: track 137.2 -> 34.6 mm
- net Picker_Motor2_E1: track 140.1 -> 51.5 mm
- net Vertical_Motor_E1: track 120.9 -> 41.9 mm
- net Motor_3_Pwm: track 78.6 -> 0.00 mm
- net M4D: track 0.00 -> 75.9 mm
- net FW4_E1: track 75.5 -> 0.00 mm
- net M1D: track 0.00 -> 74.5 mm
- net Motor_2_Pwm: track 138.1 -> 63.9 mm
- net Motor_4_DIR: track 64.1 -> 0.00 mm
- net Motor_1_DIR: track 63.4 -> 0.00 mm
- net FW3_E2: track 52.1 -> 0.00 mm
- net MPU_SCL: track 51.5 -> 0.00 mm
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Other:
- board text added: "RX"
- board text added: "TX"

Commit message: OK DONE!
Parts:
- added BT-RESTING-BED1: Conn_01x04_Female, Connector_PinHeader_2.54mm:PinHeader_2x04_P2.54mm_Vertical, F.Cu at (43.7, 103.1)
- U1: footprint Package_DIP:DIP-18_W7.62mm -> Package_DIP:DIP-16_W7.62mm_Socket
- moved GPIO_OUTPUT_PINS1 141.7 mm to (91.7, 140.0), turned to 180 degrees
- moved D3 28.6 mm to (224.5, 99.3)
- moved IMU1 21.7 mm to (219.7, 99.1)
- moved MPU1 12.7 mm to (222.5, 65.0), turned to 0 degrees
- moved GPIO_INPUT_PINS1 9.94 mm to (224.5, 72.9)
- moved pneu1 9.15 mm to (237.5, 36.3), turned to 180 degrees
- moved D4 2.70 mm to (230.6, 51.8)
- moved C1 2.52 mm to (153.4, 58.5), turned to 180 degrees
- moved D5 1.60 mm to (230.1, 40.4)
Connections:
- S1 pad 85: unconnected-(S1-Pad85) -> O5
- S1 pad 87: unconnected-(S1-Pad87) -> O4
- S1 pad 89: unconnected-(S1-Pad89) -> O3
- S1 pad 91: unconnected-(S1-Pad91) -> O2
- S1 pad 93: unconnected-(S1-Pad93) -> O1
- S2 pad 76: O1 -> unconnected-(S2-Pad76)
- S2 pad 78: FW3_E1 -> FW3_E2
- S2 pad 80: O2 -> unconnected-(S2-Pad80)
- S2 pad 82: O3 -> unconnected-(S2-Pad82)
- S2 pad 84: O4 -> unconnected-(S2-Pad84)
- S2 pad 86: O5 -> unconnected-(S2-Pad86)
- db-3 pad 10: Vertical_Motor_DIR -> GND
- db-3 pad 11: Picker_Motor1_DIR -> Horizontal_Motor_DIR
- db-3 pad 12: unconnected-(db-3-Pad12) -> Vertical_Motor_DIR
- db-3 pad 13: Picker_Motor2_E1 -> Picker_Motor1_DIR
- db-3 pad 14: Picker_Motor1_E1 -> Vertical_Motor_PWM
- db-3 pad 15: unconnected-(db-3-Pad15) -> Picker_Motor1_E1
- db-3 pad 2: unconnected-(db-3-Pad2) -> FW3_E2
- db-3 pad 3: unconnected-(db-3-Pad3) -> FW4_E1
- db-3 pad 4: unconnected-(db-3-Pad4) -> FW4_E2
- db-3 pad 5: Picker_Motor1_PWM -> Picker_Motor2_E1
- db-3 pad 6: unconnected-(db-3-Pad6) -> Vertical_Motor_E1
- db-3 pad 7: unconnected-(db-3-Pad7) -> Picker_Motor1_PWM
- db-3 pad 8: Vertical_Motor_E1 -> FW3_E1
Routing:
- net Horizontal_Motor_DIR: track 0.00 -> 140.0 mm
- net Vertical_Motor_DIR: track 0.00 -> 136.0 mm
- net Picker_Motor1_DIR: track 0.00 -> 129.8 mm
- net Vertical_Motor_PWM: track 0.00 -> 125.1 mm
- net FW3_E1: track 22.2 -> 115.8 mm
- net Picker_Motor1_E1: track 34.6 -> 118.8 mm
- net Picker_Motor1_PWM: track 38.5 -> 113.1 mm
- net Vertical_Motor_E1: track 41.9 -> 113.1 mm
- net Picker_Motor2_E1: track 51.5 -> 109.5 mm, vias 0 -> 2
- net FW3_E2: track 0.00 -> 53.5 mm
- net O3: track 0.00 -> 52.1 mm
- net O5: track 20.4 -> 62.3 mm
- net FW4_E2: track 0.00 -> 40.8 mm
- net O4: track 21.0 -> 57.2 mm
- net FW4_E1: track 0.00 -> 31.3 mm
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Other:
- board text added: "A10"
- board text added: "A14"
- board text added: "A8"
- board text added: "C10"
- board text added: "C12"
- board text added: "ST_1_BASE"
- board text removed: "B3"
- board text removed: "B5"
- board text removed: "D2"
- board text removed: "D4"
- board text removed: "D6"
- board text removed: "HMD"
- board text removed: "M3P"
- board text removed: "ST_1"
- board text removed: "VMP"
