File: ROBOT_2_PCB/ROBOT_2_PCB.kicad_sch (KiCad schematic)
At the start: 18 parts, among them J1 Conn_01x04, J2 Conn_01x02, J3 Conn_01x02, J4 DB15_Female, J5 Conn_01x01_Female, U1 ULN2003

Commit message: r2 pcb created
Parts:
- removed BT1: Conn_01x04, modfiles:bluetooth, symbol Connector_Generic:Conn_01x04
- added C1, C2: 104nF, modfiles:Capacitor_Disc_Small, symbol Device:C_Small
- added J1: Bluetooth, Connector_PinHeader_2.54mm:PinHeader_2x04_P2.54mm_Vertical, symbol Connector_Generic:Conn_02x04_Counter_Clockwise
- renumbered J1 to MPU1, J5 to NEPAL1, J2 to PN-1, J3 to PN-2, Encoders1 to db-1, J4 to db-2, DIR_PWM1 to db-3
Connections:
- net 5V: now also C1.1, C2.1, J1.1 (Pin_1), J1.2 (Pin_2); no longer MPU1.1 (Pin_1), S1.53 (5V), S1.54 (5V)
- net 5VS: now also MPU1.1 (Pin_1)
- net BT_RX: now also S1.80 (PD6), J1.7 (Pin_7), J1.8 (Pin_8); no longer S2.13 (PA3)
- net BT_TX: now also S1.79 (PD5), J1.5 (Pin_5), J1.6 (Pin_6); no longer S2.14 (PA2)
- net FW1_E1: now also db-1.5; no longer db-2.1
- net FW1_E2: now also db-1.8; no longer db-2.9 (P9)
- net FW2_E1: now also db-1.9 (P9); no longer db-2.2
- net FW2_E2: now also db-1.12 (P12); no longer db-2.10 (P10)
- net FW3_E1: now also db-1.15 (P15); no longer db-2.3
- net FW3_E2: now also db-1.14 (P14); no longer db-2.11 (P111)
- net FW4_E1: now also db-1.2; no longer db-1.1
- net FW4_E2: now also db-1.3; no longer db-2.12 (P12)
- net GND: now also S1.1 (GND), S1.49 (GND), S1.5 (GND), S1.50 (GND), S1.51 (GND), S1.52 (GND), S2.1 (GND), S2.51 (GND), S2.52 (GND), db-3.1, db-3.9 (P9), C1.2, C2.2, J1.3 (Pin_3), J1.4 (Pin_4)
- net Horizontal_Motor_DIR: now also S2.44 (PD12), db-2.1; no longer S2.93 (PA8), db-3.15 (P15)
- net Horizontal_Motor_E1: now also db-2.7; no longer db-3.2
- net Horizontal_Motor_E2: now also db-2.5
- net Horizontal_Motor_PWM: now also db-3.4; no longer db-3.7
- net MPU_SCL: now also S2.73 (PB6); no longer S1.73 (PB6)
- net MPU_SDA: now also S2.74 (PB7); no longer S1.74 (PB7)
- net Motor_1_DIR: now also S2.40 (PD8), db-2.10 (P10); no longer S1.93 (PA8)
- net Motor_1_Enc_1: now also db-1.7; no longer db-1.4
- net Motor_1_Enc_2: now also db-1.6; no longer db-1.3
- net Motor_1_Pwm: now also S2.31 (PE13), db-2.4; no longer S1.97 (PC6), db-1.10 (P10)
- net Motor_2_DIR: now also S2.14 (PA2), db-3.15 (P15); no longer S1.94 (PA9)
- net Motor_2_Enc_1: now also db-1.10 (P10); no longer S1.90 (PA15)
- net Motor_2_Enc_2: now also db-1.11 (P111); no longer db-1.7
- net Motor_2_Pwm: now also S2.32 (PE14), db-3.12 (P12); no longer S1.98 (PC7), db-1.11 (P111)
- net Motor_3_DIR: now also S2.42 (PD10), db-2.9 (P9); no longer S1.91 (PA10)
- net Motor_3_Enc_1: now also S1.97 (PC6), db-2.12 (P12); no longer S1.18 (PA6), db-1.5
- net Motor_3_Enc_2: now also db-1.13 (P13); no longer db-1.6
- net Motor_3_Pwm: now also db-2.11 (P111); no longer db-1.9 (P9)
- net Motor_4_DIR: now also S2.93 (PA8), db-3.6; no longer S1.92 (PA13)
- net Motor_4_Enc_1: now also db-1.1
- net Motor_4_Enc_2: now also db-1.4; no longer db-1.2
- net Motor_4_Pwm: now also S2.13 (PA3), db-2.14 (P14); no longer S1.96 (PC9), db-1.12 (P12)
- net Picker_Motor1_DIR: now also S2.36 (PB12), db-3.11 (P111); no longer S2.91 (PA10), db-3.14 (P14)
- net Picker_Motor1_E1: now also db-3.14 (P14); no longer db-3.10 (P10)
- net Picker_Motor1_E2: now also db-2.15 (P15); no longer db-1.14 (P14)
- net Picker_Motor1_PWM: now also db-3.5; no longer db-3.8
- net Picker_Motor2_DIR: now also S2.46 (PD14), db-2.2; no longer S2.92 (PA13), db-3.3
- net Picker_Motor2_E1: now also S2.22 (PB0), db-3.13 (P13); no longer S2.44 (PD12), db-3.1
- net Picker_Motor2_E2: now also S2.21 (PB1), db-2.8; no longer S2.45 (PD13), db-3.9 (P9)
- net Picker_Motor2_PWM: now also db-3.2; no longer db-3.5
- net Vertical_Motor_DIR: now also S2.38 (PB14), db-3.10 (P10); no longer S2.94 (PA9), db-3.4
- net Vertical_Motor_E1: now also db-3.8; no longer db-3.12 (P12)
- net Vertical_Motor_E2: now also db-2.13 (P13); no longer db-1.13 (P13)
- net Vertical_Motor_PWM: now also db-3.3; no longer db-3.6
- net I1: now reaches S2.58 (PH1)
- net I1: now also GPIO_PINS_INPUT1.1 (Pin_1)
- net I2: now reaches S2.60 (PC15)
- net I2: now also GPIO_PINS_INPUT1.2 (Pin_2)
- net I3: now reaches S2.62 (PC13)
- net I3: now also GPIO_PINS_INPUT1.3 (Pin_3)
- net I4: now reaches S2.64 (PE5)
- net I4: now also GPIO_PINS_INPUT1.4 (Pin_4)
- net I5: now reaches S2.66 (PE3)
- net I5: now also GPIO_PINS_INPUT1.5 (Pin_5)
- net O1: now reaches S2.76 (PB5)
- net O1: now also GPIO_PINS_OUTPUT1.1 (Pin_1)
- net O2: now reaches S2.78 (PB3)
- net O2: now also GPIO_PINS_OUTPUT1.2 (Pin_2)
- net O3: now reaches S2.80 (PD6)
- net O3: now also GPIO_PINS_OUTPUT1.3 (Pin_3)
- net O4: now reaches S2.82 (PD4)
- net O4: now also GPIO_PINS_OUTPUT1.4 (Pin_4)
- net O5: now reaches S2.84 (PD2)
- net O5: now also GPIO_PINS_OUTPUT1.5 (Pin_5)
- net GPIO_INPUT_1: no longer names the net of S1.38 (PB14)
- net GPIO_INPUT_1: no longer GPIO_PINS_INPUT1.1 (Pin_1)
- net GPIO_INPUT_2: no longer names the net of S1.40 (PD8)
- net GPIO_INPUT_2: no longer GPIO_PINS_INPUT1.2 (Pin_2)
- net GPIO_INPUT_3: no longer names the net of S1.42 (PD10)
- net GPIO_INPUT_3: no longer GPIO_PINS_INPUT1.3 (Pin_3)
- net GPIO_INPUT_4: no longer names the net of S1.41 (PD9)
- net GPIO_INPUT_4: no longer GPIO_PINS_INPUT1.4 (Pin_4)
- net GPIO_INPUT_5: no longer names the net of S1.43 (PD11)
- net GPIO_INPUT_5: no longer GPIO_PINS_INPUT1.5 (Pin_5)
- net GPIO_OUTPUT_1: no longer names the net of S2.41 (PD9)
- net GPIO_OUTPUT_1: no longer GPIO_PINS_OUTPUT1.1 (Pin_1)
- net GPIO_OUTPUT_2: no longer names the net of S2.43 (PD11)
- net GPIO_OUTPUT_2: no longer GPIO_PINS_OUTPUT1.2 (Pin_2)
- net GPIO_OUTPUT_3: no longer names the net of S2.47 (PD15)
- net GPIO_OUTPUT_3: no longer GPIO_PINS_OUTPUT1.3 (Pin_3)
- removed net GPIO_OUTPUT_4: GPIO_PINS_OUTPUT1.4 (Pin_4), S2.46 (PD14)
- removed net GPIO_OUTPUT_5: GPIO_PINS_OUTPUT1.5 (Pin_5), S2.42 (PD10)
Other:
- moved on the sheet: db-2

Commit message: Finally created
Parts:
- added C3: 104nF, modfiles:Capacitor_Disc_Small, symbol Device:C_Small
- added D1, D2, D3, D4, D5: LED, modfiles:LED_D3.0mm, symbol Device:LED
- added MPU1, S1I1, S2I1: 330, modfiles:Resistor_small, symbol Device:R_Small
- added pneu1, pneu2: 1K, modfiles:Resistor_small, symbol Device:R_Small
- renumbered GPIO_PINS_INPUT1 to GPIO_INPUT_PINS1, GPIO_PINS_OUTPUT1 to GPIO_OUTPUT_PINS1, MPU1 to IMU1
Connections:
- net +12V is gone; now on net 12V: PN-1.1 (Pin_1), PN-2.1 (Pin_1)
- net 12V: now also pneu1.1, pneu2.1
- net 5V: now also C3.1, S1I1.1, S2I1.1
- net 5VS: now also MPU1.1
- net GND: now also C3.2, D1.2 (A), D2.2 (A), D3.2 (A); no longer S1.49 (GND), S1.50 (GND)
- net PN_01: now also D5.2 (A)
- net PN_02: now also D4.2 (A)
- new net: D4.1 (K), pneu2.2
- new net: S1.49 (GND), S1.50 (GND)
- new net: D2.1 (K), S2I1.2
- new net: D1.1 (K), S1I1.2
- new net: D3.1 (K), MPU1.2
- new net: D5.1 (K), pneu1.2

Commit message: Finally Created1
Connections:
- net FW1_E1: now also db-1.2; no longer db-1.5
- net FW1_E2: now also db-1.5; no longer db-1.8
- net FW2_E1: now also db-1.12 (P12); no longer db-1.9 (P9)
- net FW2_E2: now also db-1.15 (P15); no longer db-1.12 (P12)
- net FW3_E1: now also db-1.6; no longer db-1.15 (P15)
- net FW3_E2: now also db-1.7; no longer db-1.14 (P14)
- net FW4_E1: now also db-1.10 (P10); no longer db-1.2
- net FW4_E2: now also db-1.9 (P9); no longer db-1.3
- net Motor_1_Enc_1: now also db-1.4; no longer db-1.7
- net Motor_1_Enc_2: now also db-1.3; no longer db-1.6
- net Motor_2_Enc_1: now also db-1.13 (P13); no longer db-1.10 (P10)
- net Motor_2_Enc_2: now also db-1.14 (P14); no longer db-1.11 (P111)
- net Motor_3_Enc_2: now also db-1.8; no longer db-1.13 (P13)
- net Motor_4_Enc_1: now also db-1.11 (P111); no longer db-1.1
- net Motor_4_Enc_2: now also db-1.1; no longer db-1.4
Changed lines of the file:
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@@
     )
   )
-  (global_label "FW3_E2" (shape input) (at 89.662 47.6504 180) (fields_autoplaced)
-    (effects (font (size 0.9 0.9)) (justify right))
-    (property "Intersheet References" "${INTERSHEET_REFS}" (id 0) (at 82.9377 47.5942 0)
+  (global_label "FW3_E2" (shape input) (at 89.662 50.1904 180) (fields_autoplaced)
+    (effects (font (size 0.9 0.9)) (justify right))
+    (property "Intersheet References" "${INTERSHEET_REFS}" (id 0) (at 82.9377 50.1342 0)
       (effects (font (size 0.9 0.9)) (justify right) hide)
     )
@@
     )
   )
-  (global_label "Motor_4_Enc_1" (shape input) (at 89.662 19.7104 180) (fields_autoplaced)
+  (global_label "Motor_4_Enc_1" (shape input) (at 89.662 32.4104 180) (fields_autoplaced)
     (effects (font (size 0.8 0.8)) (justify right))
-    (property "Intersheet References" "${INTERSHEET_REFS}" (id 0) (at 79.342 19.6604 0)
+    (property "Intersheet References" "${INTERSHEET_REFS}" (id 0) (at 79.342 32.3604 0)
       (effects (font (size 0.8 0.8)) (justify right) hide)
     )
@@
     )
   )
-  (global_label "Motor_2_Enc_1" (shape input) (at 89.662 27.3304 180) (fields_autoplaced)
-    (effects (font (size 0.9 0.9)) (justify right))
-    (property "Intersheet References" "${INTERSHEET_REFS}" (id 0) (at 78.052 27.3866 0)
+  (global_label "Motor_2_Enc_1" (shape input) (at 89.662 42.5704 180) (fields_autoplaced)
+    (effects (font (size 0.9 0.9)) (justify right))
+    (property "Intersheet References" "${INTERSHEET_REFS}" (id 0) (at 78.052 42.6266 0)
       (effects (font (size 0.9 0.9)) (justify right) hide)
     )
@@
     )
   )
-  (global_label "FW4_E2" (shape input) (at 89.662 29.8704 180) (fields_autoplaced)
-    (effects (font (size 0.9 0.9)) (justify right))
-    (property "Intersheet References" "${INTERSHEET_REFS}" (id 0) (at 82.9377 29.8142 0)
+  (global_label "FW4_E2" (shape input) (at 89.662 22.2504 180) (fields_autoplaced)
+    (effects (font (size 0.9 0.9)) (justify right))
+    (property "Intersheet References" "${INTERSHEET_REFS}" (id 0) (at 82.9377 22.1942 0)
       (effects (font (size 0.9 0.9)) (justify right) hide)
     )
@@
     )
   )
-  (global_label "FW1_E1" (shape input) (at 89.662 40.0304 180) (fields_autoplaced)
-    (effects (font (size 0.9 0.9)) (justify right))
-    (property "Intersheet References" "${INTERSHEET_REFS}" (id 0) (at 82.9377 39.9742 0)
+  (global_label "FW1_E1" (shape input) (at 89.662 24.7904 180) (fields_autoplaced)
+    (effects (font (size 0.9 0.9)) (justify right))
+    (property "Intersheet References" "${INTERSHEET_REFS}" (id 0) (at 82.9377 24.7342 0)
       (effects (font (size 0.9 0.9)) (justify right) hide)
     )
@@
     )
   )
-  (global_label "Motor_4_Enc_2" (shape input) (at 89.662 34.9504 180) (fields_autoplaced)
-    (effects (font (size 0.9 0.9)) (justify right))
-    (property "Intersheet References" "${INTERSHEET_REFS}" (id 0) (at 78.052 34.8942 0)
+  (global_label "Motor_4_Enc_2" (shape input) (at 89.662 19.7104 180) (fields_autoplaced)
+    (effects (font (size 0.9 0.9)) (justify right))
+    (property "Intersheet References" "${INTERSHEET_REFS}" (id 0) (at 78.052 19.6542 0)
       (effects (font (size 0.9 0.9)) (justify right) hide)
     )
@@
     )
   )
-  (global_label "Motor_1_Enc_2" (shape input) (at 89.662 45.1104 180) (fields_autoplaced)
-    (effects (font (size 0.9 0.9)) (justify right))
-    (property "Intersheet References" "${INTERSHEET_REFS}" (id 0) (at 78.052 45.0542 0)
+  (global_label "Motor_1_Enc_2" (shape input) (at 89.662 29.8704 180) (fields_autoplaced)
+    (effects (font (size 0.9 0.9)) (justify right))
+    (property "Intersheet References" "${INTERSHEET_REFS}" (id 0) (at 78.052 29.8142 0)
       (effects (font (size 0.9 0.9)) (justify right) hide)
     )
@@
     )
   )
-  (global_label "FW2_E1" (shape input) (at 89.662 22.2504 180) (fields_autoplaced)
-    (effects (font (size 0.9 0.9)) (justify right))
-    (property "Intersheet References" "${INTERSHEET_REFS}" (id 0) (at 82.9377 22.1942 0)
+  (global_label "FW2_E1" (shape input) (at 89.662 37.4904 180) (fields_autoplaced)
+    (effects (font (size 0.9 0.9)) (justify right))
+    (property "Intersheet References" "${INTERSHEET_REFS}" (id 0) (at 82.9377 37.4342 0)
       (effects (font (size 0.9 0.9)) (justify right) hide)
     )
@@
     )
   )
-  (global_label "Motor_1_Enc_1" (shape input) (at 89.662 50.1904 180) (fields_autoplaced)
-    (effects (font (size 0.9 0.9)) (justify right))
-    (property "Intersheet References" "${INTERSHEET_REFS}" (id 0) (at 78.052 50.1342 0)
-      (effects (font (size 0.9 0.9)) (justify right) hide)
-    )
-  )
-  (global_label "FW4_E1" (shape input) (at 89.662 24.7904 180) (fields_autoplaced)
-    (effects (font (size 0.9 0.9)) (justify right))
-    (property "Intersheet References" "${INTERSHEET_REFS}" (id 0) (at 82.9377 24.7342 0)
+  (global_label "Motor_1_Enc_1" (shape input) (at 89.662 34.9504 180) (fields_autoplaced)
+    (effects (font (size 0.9 0.9)) (justify right))
+    (property "Intersheet References" "${INTERSHEET_REFS}" (id 0) (at 78.052 34.8942 0)
+      (effects (font (size 0.9 0.9)) (justify right) hide)
+    )
+  )
+  (global_label "FW4_E1" (shape input) (at 89.662 27.3304 180) (fields_autoplaced)
+    (effects (font (size 0.9 0.9)) (justify right))
+    (property "Intersheet References" "${INTERSHEET_REFS}" (id 0) (at 82.9377 27.2742 0)
       (effects (font (size 0.9 0.9)) (justify right) hide)
     )
@@
     )
   )
-  (global_label "Motor_2_Enc_2" (shape input) (at 89.662 32.4104 180) (fields_autoplaced)
-    (effects (font (size 0.9 0.9)) (justify right))
-    (property "Intersheet References" "${INTERSHEET_REFS}" (id 0) (at 78.052 32.3542 0)
+  (global_label "Motor_2_Enc_2" (shape input) (at 89.662 47.6504 180) (fields_autoplaced)
+    (effects (font (size 0.9 0.9)) (justify right))
+    (property "Intersheet References" "${INTERSHEET_REFS}" (id 0) (at 78.052 47.5942 0)
       (effects (font (size 0.9 0.9)) (justify right) hide)
     )
@@
     )
   )
-  (global_label "FW2_E2" (shape input) (at 89.662 37.4904 180) (fields_autoplaced)
-    (effects (font (size 0.9 0.9)) (justify right))
-    (property "Intersheet References" "${INTERSHEET_REFS}" (id 0) (at 82.9377 37.4342 0)
+  (global_label "FW2_E2" (shape input) (at 89.662 52.7304 180) (fields_autoplaced)
+    (effects (font (size 0.9 0.9)) (justify right))
+    (property "Intersheet References" "${INTERSHEET_REFS}" (id 0) (at 82.9377 52.6742 0)
       (effects (font (size 0.9 0.9)) (justify right) hide)
     )
@@
     )
   )
-  (global_label "FW1_E2" (shape input) (at 89.662 55.2704 180) (fields_autoplaced)
-    (effects (font (size 0.9 0.9)) (justify right))
-    (property "Intersheet References" "${INTERSHEET_REFS}" (id 0) (at 82.9377 55.2142 0)
+  (global_label "FW1_E2" (shape input) (at 89.662 40.0304 180) (fields_autoplaced)
+    (effects (font (size 0.9 0.9)) (justify right))
+    (property "Intersheet References" "${INTERSHEET_REFS}" (id 0) (at 82.9377 39.9742 0)
       (effects (font (size 0.9 0.9)) (justify right) hide)
     )
@@
     )
   )
-  (global_label "FW3_E1" (shape input) (at 89.662 52.7304 180) (fields_autoplaced)
-    (effects (font (size 0.9 0.9)) (justify right))
-    (property "Intersheet References" "${INTERSHEET_REFS}" (id 0) (at 82.9377 52.6742 0)
+  (global_label "FW3_E1" (shape input) (at 89.662 45.1104 180) (fields_autoplaced)
+    (effects (font (size 0.9 0.9)) (justify right))
+    (property "Intersheet References" "${INTERSHEET_REFS}" (id 0) (at 82.9377 45.0542 0)
       (effects (font (size 0.9 0.9)) (justify right) hide)
     )
@@
     )
   )
-  (global_label "Motor_3_Enc_2" (shape input) (at 89.662 42.5704 180) (fields_autoplaced)
-    (effects (font (size 0.9 0.9)) (justify right))
-    (property "Intersheet References" "${INTERSHEET_REFS}" (id 0) (at 78.052 42.5142 0)
-      (effects (font (size 0.9 0.9)) (justify right) hide)
-    )
+  (global_label "Motor_3_Enc_2" (shape input) (at 89.662 55.2704 180) (fields_autoplaced)
+    (effects (font (size 0.9 0.9)) (justify right))
+    (property "Intersheet References" "${INTERSHEET_REFS}" (id 0) (at 78.052 55.2142 0)
+      (effects (font (size 0.9 0.9)) (justify right) hide)
+    )

Commit message: Redesigning in process
Connections:
- net FW1_E1: now also S1.15 (PA5), db-1.15 (P15); no longer S1.31 (PE13), db-1.2
- net FW1_E2: now also S1.78 (PB3), db-2.15 (P15); no longer S1.32 (PE14), db-1.5
- net FW2_E1: now also S1.18 (PA6), db-1.7; no longer S1.14 (PA2), db-1.12 (P12)
- net FW2_E2: now also S1.17 (PA7), db-1.8; no longer S1.13 (PA3), db-1.15 (P15)
- net FW3_E1: now also S2.15 (PA5), S2.78 (PB3); no longer S1.22 (PB0), db-1.6
- net FW3_E2: no longer S1.21 (PB1), db-1.7
- net FW4_E1: now also S2.98 (PC7); no longer S1.46 (PD14), db-1.10 (P10)
- net FW4_E2: now also S2.97 (PC6); no longer S1.47 (PD15), db-1.9 (P9)
- net Horizontal_Motor_DIR: no longer db-2.1
- net Horizontal_Motor_E1: now also db-2.5; no longer db-2.7
- net Horizontal_Motor_E2: now also db-2.4; no longer db-2.5
- net Horizontal_Motor_PWM: now also S2.31 (PE13), db-2.3; no longer S2.97 (PC6), db-3.4
- net MPU_SCL: now also S2.69 (PB8); no longer S2.73 (PB6)
- net Motor_1_Enc_1: now also db-1.5; no longer db-1.4
- net Motor_1_Enc_2: now also db-1.4; no longer db-1.3
- net Motor_1_Pwm: now also S1.31 (PE13), db-1.3; no longer S2.31 (PE13), db-2.4
- net Motor_2_Enc_1: now also db-1.12 (P12); no longer db-1.13 (P13)
- net Motor_2_Enc_2: now also db-1.13 (P13); no longer db-1.14 (P14)
- net Motor_2_Pwm: now also S1.32 (PE14), db-1.6; no longer S2.32 (PE14), db-3.12 (P12)
- net Motor_3_Enc_1: now also db-2.13 (P13); no longer db-2.12 (P12)
- net Motor_3_Enc_2: now also S1.98 (PC7), db-2.14 (P14); no longer S1.17 (PA7), db-1.8
- net Motor_3_Pwm: now also S1.14 (PA2); no longer S1.95 (PC8), db-2.11 (P111)
- net Motor_4_Enc_2: now also db-1.9 (P9); no longer db-1.1
- net Motor_4_Pwm: now also S1.13 (PA3), db-1.14 (P14); no longer S2.13 (PA3), db-2.14 (P14)
- net O2: now also S2.80 (PD6); no longer S2.78 (PB3)
- net O3: now also S2.82 (PD4); no longer S2.80 (PD6)
- net O4: now also S2.84 (PD2); no longer S2.82 (PD4)
- net O5: now also S2.86 (PD0); no longer S2.84 (PD2)
- net Picker_Motor1_E2: now also db-2.6; no longer db-2.15 (P15)
- net Picker_Motor1_PWM: now also S2.14 (PA2); no longer S2.95 (PC8)
- net Picker_Motor2_DIR: now also db-2.1; no longer db-2.2
- net Picker_Motor2_E1: now also S2.73 (PB6); no longer S2.22 (PB0)
- net Picker_Motor2_E2: now also S2.45 (PD13), db-2.2; no longer S2.21 (PB1), db-2.8
- net Picker_Motor2_PWM: now also S2.13 (PA3), db-2.7; no longer S2.96 (PC9), db-3.2
- net Vertical_Motor_E2: now also db-2.8; no longer db-2.13 (P13)
- net Vertical_Motor_PWM: now also S2.32 (PE14); no longer S2.98 (PC7), db-3.3
- net M3D: now reaches S1.41 (PD9)
- net M3D: now also db-1.2
- net M2D: now reaches S1.43 (PD11)
- net M2D: now also db-1.1
- net Motor_1_DIR: no longer names the net of S2.40 (PD8)
- net Motor_1_DIR: no longer db-2.10 (P10)
- net Motor_2_DIR: no longer names the net of db-3.15 (P15)
- net Motor_2_DIR: no longer S2.14 (PA2)
- net Motor_3_DIR: no longer names the net of S2.42 (PD10)
- net Motor_3_DIR: no longer db-2.9 (P9)
- net Motor_4_DIR: no longer names the net of S2.93 (PA8)
- net Motor_4_DIR: no longer db-3.6
- new net M1D: S1.47 (PD15), db-1.10 (P10)
- new net M4D: S1.95 (PC8), db-2.12 (P12)

Commit message: OK DONE!
Parts:
- added BT-RESTING-BED1: Conn_01x04_Female, Connector_PinHeader_2.54mm:PinHeader_2x04_P2.54mm_Vertical, symbol Connector:Conn_01x04_Female
- U1: footprint Package_DIP:DIP-18_W7.62mm -> Package_DIP:DIP-16_W7.62mm_Socket
Connections:
- net FW3_E1: now also db-3.8; no longer S2.78 (PB3)
- net FW3_E2: now also S2.78 (PB3), db-3.2
- net FW4_E1: now also db-3.3
- net FW4_E2: now also db-3.4
- net GND: now also db-3.10 (P10)
- net Horizontal_Motor_DIR: now also db-3.11 (P111)
- net O1: now also S1.93 (PA8); no longer S2.76 (PB5)
- net O2: now also S1.91 (PA10); no longer S2.80 (PD6)
- net O3: now also S1.89 (PA14); no longer S2.82 (PD4)
- net O4: now also S1.87 (PC10); no longer S2.84 (PD2)
- net O5: now also S1.85 (PC12); no longer S2.86 (PD0)
- net Picker_Motor1_DIR: now also db-3.13 (P13); no longer db-3.11 (P111)
- net Picker_Motor1_E1: now also db-3.15 (P15); no longer db-3.14 (P14)
- net Picker_Motor1_PWM: now also db-3.7; no longer db-3.5
- net Picker_Motor2_E1: now also db-3.5; no longer db-3.13 (P13)
- net Vertical_Motor_DIR: now also db-3.12 (P12); no longer db-3.10 (P10)
- net Vertical_Motor_E1: now also db-3.6; no longer db-3.8
- net Vertical_Motor_PWM: now also db-3.14 (P14)

Commit message: all file added upto this date
Connections:
- net PNEUMATIC_1: now also S2.91 (PA10); no longer S2.89 (PA14)
Changed lines of the file:
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@@
     )
   )
-  (global_label "PNEUMATIC_1" (shape input) (at 177.1396 112.3696 180) (fields_autoplaced)
+  (global_label "PNEUMATIC_1" (shape input) (at 177.1396 114.2746 180) (fields_autoplaced)
     (effects (font (size 0.9 0.9)) (justify right))
-    (property "Intersheet References" "${INTERSHEET_REFS}" (id 0) (at 166.4725 112.4258 0)
+    (property "Intersheet References" "${INTERSHEET_REFS}" (id 0) (at 166.4725 114.3308 0)
       (effects (font (size 0.9 0.9)) (justify right) hide)
     )

Commit message: Push All
Parts:
- renumbered POWER_SUPPLY1 to POW_SPLY1
Other:
- note added: "DB CONNECTION"
- note added: "EXTERNAL COMPONENT PLACEMENT"
- note added: "INDICATORS"
- note added: "MAIN CONTROLLER BOARD"
- note added: "POWER SUPPLY"
- note added: "ULN2003 FOR PNEUMATICS"
- moved on the sheet: BT-RESTING-BED1, C1, C2, C3, D1, D2, D3, D4, D5, GPIO_INPUT_PINS1, GPIO_OUTPUT_PINS1, IMU1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
