File: base_circuit/ROBOT_2_PCB.kicad_pcb (KiCad board)
At the start: 2 copper layers, 20 parts, among them J1 Conn_01x04, J2 Output_Supply, J3 Conn_01x01_Female, J4 M1,2, J5 M3,4, M1 Conn_01x04_Female, M2 Conn_01x04_Female, M3 Conn_01x04_Female, M4 Conn_01x04_Female, SW2 SW_SPDT

Commit message: Add mounting holes and clean schematic
Parts:
- added H1: MountingHole, MountingHole:MountingHole_3mm, F.Cu at (168.1, 45.0)
- added H2: MountingHole, MountingHole:MountingHole_3mm, F.Cu at (39.4, 157.7)
- added H3: MountingHole, MountingHole:MountingHole_3mm, F.Cu at (86.1, 55.6)
- added H4: MountingHole, MountingHole:MountingHole_3mm, F.Cu at (78.2, 151.4)
- added H5: MountingHole, MountingHole:MountingHole_3mm, F.Cu at (143.5, 80.3)
- added H6: MountingHole, MountingHole:MountingHole_3mm, F.Cu at (67.1, 111.5)
- added H7: MountingHole, MountingHole:MountingHole_3mm, F.Cu at (37.6, 68.8)
- added H8: MountingHole, MountingHole:MountingHole_3mm, F.Cu at (144.3, 158.2)
Connections:
- J1 pad 1: 5V -> Net-(J1-Pad1)
- J1 pad 2: 5V -> Net-(J1-Pad2)
- J1 pad 4: GND -> 5V
- S1 pad 25: (no net) -> unconnected-(S1-Pad25)
- S1 pad 26: (no net) -> unconnected-(S1-Pad26)
- S1 pad 33: (no net) -> unconnected-(S1-Pad33)
- S1 pad 34: (no net) -> unconnected-(S1-Pad34)
- S1 pad 35: (no net) -> unconnected-(S1-Pad35)
- S1 pad 36: (no net) -> unconnected-(S1-Pad36)
- S1 pad 77: (no net) -> unconnected-(S1-Pad77)

Commit message: Kam vairaxa
Parts:
- removed the D2 at (62.9, 73.7)
- removed S1I1: 330, modfiles:Resistor_small
- added C4: C_Small, modfiles:Capacitor_Disc_Small, F.Cu at (176.9, 55.0)
- added C5: C_Small, modfiles:Capacitor_Disc_Small, F.Cu at (176.9, 50.9)
- added D1: LED_Small, modfiles:LED_D3.0mm, F.Cu at (106.7, 77.9)
- added D3: LED_Small, modfiles:LED_D3.0mm, F.Cu at (84.3, 52.4)
- added D4: LED_Small, modfiles:LED_D3.0mm, F.Cu at (79.0, 52.4)
- added D5: LED_Small, modfiles:LED_D3.0mm, F.Cu at (95.8, 52.4)
- added D6: LED_Small, modfiles:LED_D3.0mm, F.Cu at (89.9, 52.4)
- added D7: LED_Small, modfiles:LED_D3.0mm, F.Cu at (73.0, 91.3)
- added F1: Fuse_Small, modfiles:Fuse_Holder, F.Cu at (86.9, 62.7)
- added J6: Conn_01x02_Male, modfiles:Connector_Bornier_2, F.Cu at (192.9, 55.2)
- added J7: Conn_01x02_Male, modfiles:Connector_Bornier_2, F.Cu at (192.9, 44.7)
- added R1: R_Small, modfiles:Resistor_small, F.Cu at (137.9, 61.5)
- added R2: R_Small, modfiles:Resistor_small, F.Cu at (137.7, 66.8)
- added R3: R_Small, modfiles:Resistor_small, F.Cu at (137.9, 51.8)
- added R4: R_Small, modfiles:Resistor_small, F.Cu at (137.9, 56.6)
- added R5: R_Small, modfiles:Resistor_small, F.Cu at (150.1, 63.8)
- added R6: R_Small, modfiles:Resistor_small, F.Cu at (137.4, 71.4)
- J2: value Output_Supply -> Conn_01x02_Male; footprint modfiles:JST_5_BIG -> modfiles:Connector_Bornier_2
- moved H4 143.8 mm to (203.3, 80.4)
- moved H6 141.2 mm to (182.6, 30.4)
- moved H7 109.7 mm to (114.7, 146.9)
- moved H2 99.8 mm to (98.4, 77.2)
- moved H5 76.4 mm to (182.3, 146.1)
- moved H8 71.8 mm to (73.3, 147.1)
- moved C2 43.3 mm to (184.1, 77.3), turned to 180 degrees
- moved M3 43.0 mm to (87.0, 137.4), turned to 0 degrees
- moved J2 42.2 mm to (192.9, 65.8), turned to 90 degrees
- moved POW_SPLY1 41.2 mm to (82.4, 42.9)
- moved M2 41.0 mm to (86.9, 131.5), turned to 0 degrees
- moved S1 39.7 mm to (142.2, 89.4)
- moved IMU1 39.0 mm to (189.0, 78.5), turned to 0 degrees
- moved J4 38.2 mm to (194.8, 132.1)
- moved J5 37.6 mm to (193.3, 103.9)
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- renumbered D3 to D2
Connections:
- C1 pad 1: 3.3V -> VDD
- D2 pad 1: Net-(D3-Pad1) -> GND
- D2 pad 2: GND -> Net-(D2-Pad2)
- MPU1 pad 2: Net-(D3-Pad1) -> Net-(D2-Pad2)
- S1 pad 11: Motor_2_Enc_2 -> Motor_1_Enc_2
- S1 pad 12: Motor_2_Enc_1 -> Motor_1_Enc_1
- S1 pad 2: unconnected-(S1-Pad2) -> GND
- S1 pad 27: Motor_1_Enc_1 -> Motor_2_Enc_1
- S1 pad 29: Motor_1_Enc_2 -> Motor_2_Enc_2
- S1 pad 3: 3.3V -> VDD
- S1 pad 4: 3.3V -> VDD
- S1 pad 44: Motor_4_Enc_1 -> Motor_3_Enc_1
- S1 pad 45: Motor_4_Enc_2 -> Motor_3_Enc_2
- S1 pad 51: unconnected-(S1-Pad51) -> GND
- S1 pad 97: Motor_3_Enc_1 -> Motor_4_Enc_1
- S1 pad 98: Motor_3_Enc_2 -> Motor_4_Enc_2
Routing:
- net GND: track 497.5 -> 2.54 mm, vias 2 -> 0
- net 5V: track 351.4 -> 30.4 mm
- net Motor_4_Pwm: track 121.0 -> 0.00 mm
- net TX: track 120.2 -> 14.6 mm
- net 3.3V: track 150.9 -> 47.1 mm
- net RX: track 125.2 -> 23.8 mm
- net Motor_3_Enc_2: track 115.4 -> 23.9 mm
- net Motor_3_Pwm: track 85.2 -> 0.00 mm
- net M3D: track 82.0 -> 0.00 mm
- net M2D: track 81.2 -> 0.00 mm
- net Motor_3_Enc_1: track 120.5 -> 42.3 mm
- net Net-(D4-Pad1): track 0.00 -> 64.6 mm
- net Motor_4_Enc_2: track 19.9 -> 84.4 mm
- net SDA: track 60.7 -> 0.00 mm
- net SCL: track 56.0 -> 0.00 mm
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Other:
- board text added: "12 5A 5V 3V3 G"
- board text added: "5 G SCL SDA"
- board text added: "GND"
- board text removed: "12V"
- board text removed: "3.3V"
- board text removed: "5"
- board text removed: "5A"
- board text removed: "G"
- board text removed: "OUT_POWER"
- board text removed: "SCL"
- board text removed: "SDA"
