File: walkie_talkie/walkie_talkie.kicad_sch (KiCad schematic)
At the start: 18 parts, among them J1 Conn_01x02, Q1 2N3904, SW1 SW_Push_Dual, U1 NRF24L01_Breakout, U2 MicroPhone, U3 L7805

Commit message: rewiring
Parts:
- SW1: footprint Button_Switch_THT:SW_PUSH-12mm -> modFilesUpdated:tactile_push_button
Changed lines of the file:
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@@
       (effects (font (size 1.27 1.27)))
     )
-    (property "Footprint" "Button_Switch_THT:SW_PUSH-12mm" (at 37.465 66.04 0)
+    (property "Footprint" "modFilesUpdated:tactile_push_button" (at 37.465 66.04 0)
       (effects (font (size 1.27 1.27)) hide)
     )
