File: bluepill-Encoder-Comm/bluepill-Encoder-Comm.kicad_pcb (KiCad board)
At the start: 2 copper layers, 38 parts, among them J1 Conn_01x05, J10 Conn_02x05_Counter_Clockwise, J11 Conn_01x02_Pin, J7 Conn_01x02_Pin, J8 Conn_01x04, J9 Conn_02x05_Counter_Clockwise, Q1 TIP122, Q2 TIP122, U3 Buck

Commit message: Modified necessary designs in PCB
Parts:
- removed J1: Conn_01x05, modFiles:JST_5_BIG
- removed J10, J9: Conn_02x05_Counter_Clockwise, modFiles:bluetooth
- added 1K: R, modFiles:Resistor_small, F.Cu at (138.6, 132.9)
- added D2: D_Small, modFiles:Diode_Medium, F.Cu at (85.3, 83.2)
- added J2: Conn_01x02_Pin, modFiles:Solar_Connector, F.Cu at (180.2, 71.5)
- added J3: Conn_01x04_Pin, modFiles:Barrier_Terminal_Block, F.Cu at (34.1, 134.4)
- added J4: Conn_01x04_Pin, modFiles:Barrier_Terminal_Block, F.Cu at (34.1, 132.2)
- added J5: Conn_02x03_Odd_Even, modFiles:current sensor, F.Cu at (196.2, 133.5)
- added R3: 1K, modFiles:Resistor_small, F.Cu at (143.4, 126.7)
- added U1: SIM800L-CORE, sim800l:SIM800L-CORE, F.Cu at (43.9, 70.7)
- R1: value R_Small -> 5; footprint modFiles:Voltage_Regulators -> modFiles:Resistor_small
- R2: value 1k -> 1K
- R4: value 2k -> 2K
- R6, R7, R8: value R_Small -> 220
- Rly1: footprint modFiles:Relay_6V -> modFiles:Relay_HLS_MEDIUM
- Rly2: footprint modFiles:Diode_Medium -> modFiles:Relay_HLS_MEDIUM
- moved J11 118.0 mm to (191.6, 147.1)
- moved D4 108.0 mm to (171.4, 140.7)
- moved D10 100.9 mm to (91.1, 155.8), turned to 90 degrees
- moved C5 100.8 mm to (46.4, 62.8)
- moved D8 98.5 mm to (96.2, 155.8), turned to 90 degrees
- moved R5 98.4 mm to (192.5, 67.0), turned to 90 degrees
- moved D11 97.2 mm to (86.0, 155.8), turned to 90 degrees
- moved R6 95.7 mm to (178.5, 133.1), turned to -90 degrees
- moved D9 92.2 mm to (101.3, 155.8), turned to 90 degrees
- moved Rly1 87.0 mm to (193.5, 102.0)
- moved D5 87.0 mm to (139.6, 142.2), turned to 180 degrees
- moved U3 85.6 mm to (107.2, 120.8), turned to 90 degrees
- moved C6 77.5 mm to (61.5, 103.2), turned to -90 degrees
- moved J7 69.8 mm to (125.0, 136.4)
- moved C4 67.1 mm to (78.9, 68.7), turned to 90 degrees
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Connections:
- A2 pad 16: unconnected-(A2-D13-Pad16) -> /I3
- A2 pad 17: unconnected-(A2-3V3-Pad17) -> /I1
- A2 pad 18: unconnected-(A2-AREF-Pad18) -> /I2
- A2 pad 19: unconnected-(A2-A0-Pad19) -> /UPPER2
- A2 pad 2: unconnected-(A2-D0/RX-Pad2) -> /RING
- A2 pad 20: unconnected-(A2-A1-Pad20) -> /UPPER1
- A2 pad 21: unconnected-(A2-A2-Pad21) -> /LOWER1
- A2 pad 22: unconnected-(A2-A3-Pad22) -> /LOWER2
- A2 pad 23: unconnected-(A2-A4-Pad23) -> /RELAY1
- A2 pad 24: unconnected-(A2-A5-Pad24) -> /RELAY2
- A2 pad 30: +10V -> /10V_regulated
- D1 pad 2: GND -> /R1_GND
- D3 pad 2: GND -> /R2_GND
- D4 pad 1: GND -> GND1
- J11 pad 2: GND -> GND1
- Q1 pad 1: /Relay1 -> Net-(Q1-B)
- Q2 pad 1: /Relay2 -> Net-(Q2-B)
- Rly1 pad 1: /R1_GND -> /+48V_I
- Rly1 pad 2: /M+ -> +12V
- Rly2 pad 1: /R2_GND -> /+48V_I
- Rly2 pad 2: /M- -> +12V
Routing:
- net +5V: track 0.00 -> 529.1 mm
- net +12V: track 0.00 -> 243.0 mm
- net /RELAY1: track 0.00 -> 122.8 mm
- net GND: track 0.00 -> 120.6 mm
- net /RELAY2: track 0.00 -> 116.8 mm
- net +4V: track 0.00 -> 103.5 mm
- net /LOWER2: track 0.00 -> 87.9 mm
- net /LOWER1: track 0.00 -> 84.4 mm
- net /GSM_TX: track 0.00 -> 70.2 mm
- net /M-: track 0.00 -> 62.0 mm
- net /+48V_I: track 0.00 -> 61.7 mm
- net /UPPER2: track 0.00 -> 57.9 mm
- net Net-(Q1-B): track 0.00 -> 49.6 mm
- net /M+: track 0.00 -> 47.9 mm
- net /UPPER1: track 0.00 -> 45.3 mm
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- added copper zone on B.Cu, net GND
- added copper zone on B.Cu, net GND1
Other:
- board text added: "10V GND"
- board text added: "12V"
- board text added: "12V GND"
- board text added: "12V GND BUCK_IN"
- board text added: "48V GND1"
- board text added: "4V"
- board text added: "4V GND"
- board text added: "5V"
- board text added: "5V GND C1 C2"
- board text added: "BUCK_OUT GND 4V"
- board text added: "DTR"
- board text added: "GND"
- board text added: "GND R2_GND RELAY1"
- board text added: "GSM_RX"
- board text added: "GSM_TX"
- board text added: "LOWER1"
- board text added: "LOWER2"
- board text added: "M+"
- board text added: "M-"
- board text added: "OUTPUT M- M+"
- board text added: "R1_GND"
- board text added: "RING"
- board text added: "RST"
- board text added: "UPPER1"
- board text added: "UPPER2"
