File: bluepill-Encoder-Comm/bluepill-Encoder-Comm.kicad_sch (KiCad schematic)
At the start: 39 parts, among them J1 Conn_01x05, J10 Conn_02x05_Counter_Clockwise, J11 Conn_01x02_Pin, J7 Conn_01x02_Pin, J8 Conn_01x04, J9 Conn_02x05_Counter_Clockwise, Q1 TIP122, Q2 TIP122, U3 Buck

Commit message: Modified necessary designs in PCB
Parts:
- removed J1: Conn_01x05, modFiles:JST_5_BIG, symbol Connector_Generic:Conn_01x05
- removed J10, J9: Conn_02x05_Counter_Clockwise, modFiles:bluetooth, symbol Connector_Generic:Conn_02x05_Counter_Clockwise
- added J2: Conn_01x02_Pin, modFiles:Solar_Connector, symbol Connector:Conn_01x02_Pin
- added J3, J4: Conn_01x04_Pin, modFiles:Barrier_Terminal_Block, symbol Connector:Conn_01x04_Pin
- added J5: Conn_02x03_Odd_Even, modFiles:current sensor, symbol Connector_Generic:Conn_02x03_Odd_Even
- added R14, R3: R, modFiles:Resistor_small, symbol Device:R
- added U1: SIM800L-CORE, sim800l:SIM800L-CORE, symbol sim800l-core:SIM800L-CORE
- D2: footprint (none) -> modFiles:Diode_Medium
- R1: footprint modFiles:Voltage_Regulators -> modFiles:Resistor_small
- Rly1: footprint modFiles:Relay_6V -> modFiles:Relay_HLS_MEDIUM
- Rly2: footprint modFiles:Diode_Medium -> modFiles:Relay_HLS_MEDIUM
Connections:
- net +48V: now also J5.1 (Pin_1); no longer Rly1.3, Rly2.3
- net +4V: now also U1.2 (VCC)
- net +5V: now also J3.4 (Pin_4), J4.4 (Pin_4), J5.2 (Pin_2)
- net DTR: now also U1.11 (DTR)
- net GND: now also J3.3 (Pin_3), J4.3 (Pin_3), J5.6 (Pin_6), U1.6 (GND); no longer A2.4 (GND), D4.1 (K), J11.2 (Pin_2), Rly1.4, Rly2.4
- net GSM_RX: now also U1.4 (RXD)
- net GSM_TX: now also U1.5 (TXD)
- net LOWER1: now also A2.21 (A2), J4.2 (Pin_2); no longer A2.22 (A3)
- net LOWER2: now also A2.22 (A3), J4.1 (Pin_1); no longer A2.21 (A2)
- net M+: now also J2.1 (Pin_1)
- net M-: now also J2.2 (Pin_2)
- net RING: now also U1.12 (RING)
- net RST: now also U1.3 (RST)
- net UPPER1: now also J3.1 (Pin_1)
- net UPPER2: now also J3.2 (Pin_2)
- net RELAY1: now reaches A2.23 (A4)
- net RELAY1: now also R3.1
- net RELAY2: now reaches A2.24 (A5)
- net RELAY2: now also R14.1
- net Relay1: no longer names the net of Q1.1 (B)
- net Relay1: now also R3.2
- net Relay2: no longer names the net of Q2.1 (B)
- net Relay2: now also R14.2
- new net +48V_I: J5.3 (Pin_3), Rly1.4, Rly2.4
- new net GND1: D4.1 (K), J11.2 (Pin_2), Rly1.3, Rly2.3
- new net OUT: J5.4 (Pin_4)
Other:
- moved on the sheet: R1
